Commit message: Replaced spherical joints with 3 rotations, added collision hulls and other missing files required by mc_rtc

File: urdf/human_with_articulated_hands.urdf (robot description, URDF)
Before this commit: robot HUMAN, 62 links, 61 joints
Joints:
- joint LHandBabyLink1: axis (none) -> -1 0 0; limit (none) -> lower=0.0 upper=1.57 effort=1 velocity=1; type fixed -> revolute
- joint LHandBabyLink2: axis (none) -> -1 0 0; limit (none) -> lower=0.0 upper=1.57 effort=1 velocity=1; type fixed -> revolute
- joint LHandBabyLink3: axis (none) -> -1 0 0; limit (none) -> lower=0.0 upper=1.57 effort=1 velocity=1; type fixed -> revolute
- joint LHandIndexLink1: axis (none) -> -1 0 0; limit (none) -> lower=0.0 upper=1.57 effort=1 velocity=1; type fixed -> revolute
- joint LHandIndexLink2: axis (none) -> -1 0 0; limit (none) -> lower=0.0 upper=1.57 effort=1 velocity=1; type fixed -> revolute
- joint LHandIndexLink3: axis (none) -> -1 0 0; limit (none) -> lower=0.0 upper=1.57 effort=1 velocity=1; type fixed -> revolute
- joint LHandMiddleLink1: axis (none) -> -1 0 0; limit (none) -> lower=0.0 upper=1.57 effort=1 velocity=1; type fixed -> revolute
- joint LHandMiddleLink2: axis (none) -> -1 0 0; limit (none) -> lower=0.0 upper=1.57 effort=1 velocity=1; type fixed -> revolute
- joint LHandMiddleLink3: axis (none) -> -1 0 0; limit (none) -> lower=0.0 upper=1.57 effort=1 velocity=1; type fixed -> revolute
- joint LHandRingLink1: axis (none) -> -1 0 0; limit (none) -> lower=0.0 upper=1.57 effort=1 velocity=1; type fixed -> revolute
- joint LHandRingLink2: axis (none) -> -1 0 0; limit (none) -> lower=0.0 upper=1.57 effort=1 velocity=1; type fixed -> revolute
- joint LHandRingLink3: axis (none) -> -1 0 0; limit (none) -> lower=0.0 upper=1.57 effort=1 velocity=1; type fixed -> revolute
- joint LHandThumbLink1: axis (none) -> 0 1 0; limit (none) -> lower=0.0 upper=1.57 effort=1 velocity=1; origin xyz=0.02 0.016 -0.016 rpy=0.0 0.2 0.9 -> xyz=0.02 0.016 -0.016 rpy=0.0 0.0 0.0; type fixed -> revolute
- joint LHandThumbLink2: axis (none) -> 0 1 0; limit (none) -> lower=0.0 upper=1.57 effort=1 velocity=1; type fixed -> revolute
- joint LHandThumbLink3: axis (none) -> 0 1 0; limit (none) -> lower=0.0 upper=1.57 effort=1 velocity=1; type fixed -> revolute
- joint RHandBabyLink1: axis (none) -> -1 0 0; limit (none) -> lower=0.0 upper=1.57 effort=1 velocity=1; type fixed -> revolute
- joint RHandBabyLink2: axis (none) -> -1 0 0; limit (none) -> lower=0.0 upper=1.57 effort=1 velocity=1; type fixed -> revolute
- joint RHandBabyLink3: axis (none) -> -1 0 0; limit (none) -> lower=0.0 upper=1.57 effort=1 velocity=1; type fixed -> revolute
- joint RHandIndexLink1: axis (none) -> -1 0 0; limit (none) -> lower=0.0 upper=1.57 effort=1 velocity=1; type fixed -> revolute
- joint RHandIndexLink2: axis (none) -> -1 0 0; limit (none) -> lower=0.0 upper=1.57 effort=1 velocity=1; type fixed -> revolute
- joint RHandIndexLink3: axis (none) -> -1 0 0; limit (none) -> lower=0.0 upper=1.57 effort=1 velocity=1; type fixed -> revolute
- joint RHandMiddleLink1: axis (none) -> -1 0 0; limit (none) -> lower=0.0 upper=1.57 effort=1 velocity=1; type fixed -> revolute
- joint RHandMiddleLink2: axis (none) -> -1 0 0; limit (none) -> lower=0.0 upper=1.57 effort=1 velocity=1; type fixed -> revolute
- joint RHandMiddleLink3: axis (none) -> -1 0 0; limit (none) -> lower=0.0 upper=1.57 effort=1 velocity=1; type fixed -> revolute
- joint RHandRingLink1: axis (none) -> -1 0 0; limit (none) -> lower=0.0 upper=1.57 effort=1 velocity=1; type fixed -> revolute
- joint RHandRingLink2: axis (none) -> -1 0 0; limit (none) -> lower=0.0 upper=1.57 effort=1 velocity=1; type fixed -> revolute
- joint RHandRingLink3: axis (none) -> -1 0 0; limit (none) -> lower=0.0 upper=1.57 effort=1 velocity=1; type fixed -> revolute
- joint RHandThumbLink0: axis (none) -> 0 1 0; limit (none) -> lower=0.0 upper=1.57 effort=1 velocity=1; origin xyz=0.02 -0.016 -0.016 rpy=0.0 0.2 -0.9 -> xyz=0.02 -0.016 -0.016 rpy=0.0 0.0 0.0; type fixed -> revolute
- joint RHandThumbLink1: axis (none) -> 0 1 0; limit (none) -> lower=0.0 upper=1.57 effort=1 velocity=1; type fixed -> revolute
- joint RHandThumbLink2: axis (none) -> 0 1 0; limit (none) -> lower=0.0 upper=1.57 effort=1 velocity=1; type fixed -> revolute
