Commit message: Removed fingers completely from the main URDF, added seperate urdf with fixed fingers, added inertia parameters for auxiliary links for spherical joints

File: urdf/human_with_fixed_fingers.urdf (robot description, URDF)
Before this commit: robot HUMAN, 32 links, 31 joints
Links:
- added link LHandBaby1Link, mass 0.0182; collision mesh filename=package://human_description/meshes/LBaby1stPhalange.dae; visual mesh filename=package://human_description/meshes/LBaby1stPhalange.dae
- added link LHandBaby2Link, mass 0.0182; collision mesh filename=package://human_description/meshes/LBaby2ndPhalange.dae; visual mesh filename=package://human_description/meshes/LBaby2ndPhalange.dae
- added link LHandBaby3Link, mass 0.0182; collision mesh filename=package://human_description/meshes/LBaby3rdPhalange.dae; visual mesh filename=package://human_description/meshes/LBaby3rdPhalange.dae
- added link LHandIndex1Link, mass 0.0182; collision mesh filename=package://human_description/meshes/LIndex1stPhalange.dae; visual mesh filename=package://human_description/meshes/LIndex1stPhalange.dae
- added link LHandIndex2Link, mass 0.0182; collision mesh filename=package://human_description/meshes/LIndex2ndPhalange.dae; visual mesh filename=package://human_description/meshes/LIndex2ndPhalange.dae
- added link LHandIndex3Link, mass 0.0182; collision mesh filename=package://human_description/meshes/LIndex3rdPhalange.dae; visual mesh filename=package://human_description/meshes/LIndex3rdPhalange.dae
- added link LHandMiddle1Link, mass 0.0182; collision mesh filename=package://human_description/meshes/LMiddle1stPhalange.dae; visual mesh filename=package://human_description/meshes/LMiddle1stPhalange.dae
- added link LHandMiddle2Link, mass 0.0182; collision mesh filename=package://human_description/meshes/LMiddle2ndPhalange.dae; visual mesh filename=package://human_description/meshes/LMiddle2ndPhalange.dae
- added link LHandMiddle3Link, mass 0.0182; collision mesh filename=package://human_description/meshes/LMiddle3rdPhalange.dae; visual mesh filename=package://human_description/meshes/LMiddle3rdPhalange.dae
- added link LHandRing1Link, mass 0.0182; collision mesh filename=package://human_description/meshes/LRing1stPhalange.dae; visual mesh filename=package://human_description/meshes/LRing1stPhalange.dae
- added link LHandRing2Link, mass 0.0182; collision mesh filename=package://human_description/meshes/LRing2ndPhalange.dae; visual mesh filename=package://human_description/meshes/LRing2ndPhalange.dae
- added link LHandRing3Link, mass 0.0182; collision mesh filename=package://human_description/meshes/LRing3rdPhalange.dae; visual mesh filename=package://human_description/meshes/LRing3rdPhalange.dae
- added link LHandThumb0Link, mass 0.0182; collision mesh filename=package://human_description/meshes/LThumb0thPhalange.dae; visual mesh filename=package://human_description/meshes/LThumb0thPhalange.dae
- added link LHandThumb1Link, mass 0.0182; collision mesh filename=package://human_description/meshes/LThumb1stPhalange.dae; visual mesh filename=package://human_description/meshes/LThumb1stPhalange.dae
- added link LHandThumb2Link, mass 0.0182; collision mesh filename=package://human_description/meshes/LThumb2ndPhalange.dae; visual mesh filename=package://human_description/meshes/LThumb2ndPhalange.dae
- added link RHandBaby1Link, mass 0.0182; collision mesh filename=package://human_description/meshes/RBaby1stPhalange.dae; visual mesh filename=package://human_description/meshes/RBaby1stPhalange.dae
- added link RHandBaby2Link, mass 0.0182; collision mesh filename=package://human_description/meshes/RBaby2ndPhalange.dae; visual mesh filename=package://human_description/meshes/RBaby2ndPhalange.dae
- added link RHandBaby3Link, mass 0.0182; collision mesh filename=package://human_description/meshes/RBaby3rdPhalange.dae; visual mesh filename=package://human_description/meshes/RBaby3rdPhalange.dae
- added link RHandIndex1Link, mass 0.0182; collision mesh filename=package://human_description/meshes/RIndex1stPhalange.dae; visual mesh filename=package://human_description/meshes/RIndex1stPhalange.dae
- added link RHandIndex2Link, mass 0.0182; collision mesh filename=package://human_description/meshes/RIndex2ndPhalange.dae; visual mesh filename=package://human_description/meshes/RIndex2ndPhalange.dae
- added link RHandIndex3Link, mass 0.0182; collision mesh filename=package://human_description/meshes/RIndex3rdPhalange.dae; visual mesh filename=package://human_description/meshes/RIndex3rdPhalange.dae
- added link RHandMiddle1Link, mass 0.0182; collision mesh filename=package://human_description/meshes/RMiddle1stPhalange.dae; visual mesh filename=package://human_description/meshes/RMiddle1stPhalange.dae
- added link RHandMiddle2Link, mass 0.0182; collision mesh filename=package://human_description/meshes/RMiddle2ndPhalange.dae; visual mesh filename=package://human_description/meshes/RMiddle2ndPhalange.dae
- added link RHandMiddle3Link, mass 0.0182; collision mesh filename=package://human_description/meshes/RMiddle3rdPhalange.dae; visual mesh filename=package://human_description/meshes/RMiddle3rdPhalange.dae
- added link RHandRing1Link, mass 0.0182; collision mesh filename=package://human_description/meshes/RRing1stPhalange.dae; visual mesh filename=package://human_description/meshes/RRing1stPhalange.dae
- added link RHandRing2Link, mass 0.0182; collision mesh filename=package://human_description/meshes/RRing2ndPhalange.dae; visual mesh filename=package://human_description/meshes/RRing2ndPhalange.dae
- added link RHandRing3Link, mass 0.0182; collision mesh filename=package://human_description/meshes/RRing3rdPhalange.dae; visual mesh filename=package://human_description/meshes/RRing3rdPhalange.dae
- added link RHandThumb0Link, mass 0.0182; collision mesh filename=package://human_description/meshes/RThumb0thPhalange.dae; visual mesh filename=package://human_description/meshes/RThumb0thPhalange.dae
- added link RHandThumb1Link, mass 0.0182; collision mesh filename=package://human_description/meshes/RThumb1stPhalange.dae; visual mesh filename=package://human_description/meshes/RThumb1stPhalange.dae
- added link RHandThumb2Link, mass 0.0182; collision mesh filename=package://human_description/meshes/RThumb2ndPhalange.dae; visual mesh filename=package://human_description/meshes/RThumb2ndPhalange.dae
Joints:
- added joint LHandBabyLink1: type fixed, parent LHandLink, child LHandBaby1Link, origin xyz=-0.015 0.079 -0.022 rpy=0.0 0.0 0.0
- added joint LHandBabyLink2: type fixed, parent LHandBaby1Link, child LHandBaby2Link, origin xyz=-0.0 0.02 0.0 rpy=0.0 0.0 0.0
- added joint LHandBabyLink3: type fixed, parent LHandBaby2Link, child LHandBaby3Link, origin xyz=-0.0 0.02 0.0 rpy=0.0 0.0 0.0
- added joint LHandIndexLink1: type fixed, parent LHandLink, child LHandIndex1Link, origin xyz=0.0425 0.078 -0.01 rpy=0.0 0.0 0.0
- added joint LHandIndexLink2: type fixed, parent LHandIndex1Link, child LHandIndex2Link, origin xyz=-0.0 0.035 0.0 rpy=0.0 0.0 0.0
- added joint LHandIndexLink3: type fixed, parent LHandIndex2Link, child LHandIndex3Link, origin xyz=-0.0 0.022 0.0 rpy=0.0 0.0 0.0
- added joint LHandMiddleLink1: type fixed, parent LHandLink, child LHandMiddle1Link, origin xyz=0.02 0.09 -0.01 rpy=0.0 0.0 0.0
- added joint LHandMiddleLink2: type fixed, parent LHandMiddle1Link, child LHandMiddle2Link, origin xyz=-0.0 0.028 0.0 rpy=0.0 0.0 0.0
- added joint LHandMiddleLink3: type fixed, parent LHandMiddle2Link, child LHandMiddle3Link, origin xyz=-0.0 0.025 0.0 rpy=0.0 0.0 0.0
- added joint LHandRingLink1: type fixed, parent LHandLink, child LHandRing1Link, origin xyz=-0.001 0.085 -0.01 rpy=0.0 0.0 0.0
- added joint LHandRingLink2: type fixed, parent LHandRing1Link, child LHandRing2Link, origin xyz=-0.0 0.0225 0.0 rpy=0.0 0.0 0.0
- added joint LHandRingLink3: type fixed, parent LHandRing2Link, child LHandRing3Link, origin xyz=-0.0 0.028 0.0 rpy=0.0 0.0 0.0
- added joint LHandThumbLink1: type fixed, parent LHandLink, child LHandThumb0Link, origin xyz=0.02 0.016 -0.016 rpy=0.0 0.2 0.9
- added joint LHandThumbLink2: type fixed, parent LHandThumb0Link, child LHandThumb1Link, origin xyz=0.045 0.0 0.0 rpy=0.0 0.0 0.0
- added joint LHandThumbLink3: type fixed, parent LHandThumb1Link, child LHandThumb2Link, origin xyz=0.026 0.0 0.0 rpy=0.0 0.0 0.0
- added joint RHandBabyLink1: type fixed, parent RHandLink, child RHandBaby1Link, origin xyz=-0.015 -0.079 -0.022 rpy=0.0 0.0 0.0
- added joint RHandBabyLink2: type fixed, parent RHandBaby1Link, child RHandBaby2Link, origin xyz=-0.0 -0.02 0.0 rpy=0.0 0.0 0.0
- added joint RHandBabyLink3: type fixed, parent RHandBaby2Link, child RHandBaby3Link, origin xyz=-0.0 -0.02 0.0 rpy=0.0 0.0 0.0
- added joint RHandIndexLink1: type fixed, parent RHandLink, child RHandIndex1Link, origin xyz=0.0425 -0.078 -0.01 rpy=0.0 0.0 0.0
- added joint RHandIndexLink2: type fixed, parent RHandIndex1Link, child RHandIndex2Link, origin xyz=-0.0 -0.035 0.0 rpy=0.0 0.0 0.0
- added joint RHandIndexLink3: type fixed, parent RHandIndex2Link, child RHandIndex3Link, origin xyz=-0.0 -0.022 0.0 rpy=0.0 0.0 0.0
- added joint RHandMiddleLink1: type fixed, parent RHandLink, child RHandMiddle1Link, origin xyz=0.02 -0.09 -0.01 rpy=0.0 0.0 0.0
- added joint RHandMiddleLink2: type fixed, parent RHandMiddle1Link, child RHandMiddle2Link, origin xyz=-0.0 -0.028 0.0 rpy=0.0 0.0 0.0
- added joint RHandMiddleLink3: type fixed, parent RHandMiddle2Link, child RHandMiddle3Link, origin xyz=-0.0 -0.025 0.0 rpy=0.0 0.0 0.0
- added joint RHandRingLink1: type fixed, parent RHandLink, child RHandRing1Link, origin xyz=-0.001 -0.085 -0.01 rpy=0.0 0.0 0.0
- added joint RHandRingLink2: type fixed, parent RHandRing1Link, child RHandRing2Link, origin xyz=-0.0 -0.0225 0.0 rpy=0.0 0.0 0.0
- added joint RHandRingLink3: type fixed, parent RHandRing2Link, child RHandRing3Link, origin xyz=-0.0 -0.028 0.0 rpy=0.0 0.0 0.0
- added joint RHandThumbLink0: type fixed, parent RHandLink, child RHandThumb0Link, origin xyz=0.02 -0.016 -0.016 rpy=0.0 0.2 -0.9
- added joint RHandThumbLink1: type fixed, parent RHandThumb0Link, child RHandThumb1Link, origin xyz=0.045 0.0 0.0 rpy=0.0 0.0 0.0
- added joint RHandThumbLink2: type fixed, parent RHandThumb1Link, child RHandThumb2Link, origin xyz=0.026 0.0 0.0 rpy=0.0 0.0 0.0
