Commit message: More contact surfaces, additional ankle joint, minor URDF fixes

File: urdf/human.urdf (robot description, URDF)
Before this commit: robot HUMAN, 32 links, 31 joints
Links:
- added link shin2lankle_1, mass 0.2; collision sphere radius=0.02; visual sphere radius=0.02
- added link shin2rankle_1, mass 0.2; collision sphere radius=0.02; visual sphere radius=0.02
Joints:
- added joint LAnkle_1: type revolute, parent shin2lankle_1, child LAnkleLink, origin xyz=0.0 0.0 0.0 rpy=0.0 0.0 0.0, axis 1 0 0, limit lower=-0.5 upper=0.5 effort=100 velocity=100
- added joint RAnkle_1: type revolute, parent shin2rankle_1, child RAnkleLink, origin xyz=0.0 0.0 0.0 rpy=0.0 0.0 0.0, axis 1 0 0, limit lower=-0.5 upper=0.5 effort=100 velocity=100
- joint Head_0: limit lower=-0.62 upper=0.62 effort=1 velocity=1 -> lower=-0.62 upper=0.62 effort=100 velocity=100
- joint Head_1: limit lower=-0.45 upper=0.45 effort=1 velocity=1 -> lower=-0.45 upper=0.45 effort=100 velocity=100
- joint Head_2: limit lower=-1.1 upper=1.1 effort=1 velocity=1 -> lower=-1.1 upper=1.1 effort=100 velocity=100
- joint LAnkle_0: child LAnkleLink -> shin2lankle_1; limit lower=-0.78 upper=1.3 effort=1 velocity=1 -> lower=-0.78 upper=1.3 effort=100 velocity=100
- joint LArm_0: limit lower=-1.42 upper=1.57 effort=1 velocity=1 -> lower=-1.42 upper=1.57 effort=100 velocity=100
- joint LArm_1: limit lower=-1.2 upper=1.2 effort=1 velocity=1 -> lower=-1.2 upper=1.2 effort=100 velocity=100
- joint LArm_2: limit lower=-2.25 upper=0.78 effort=1 velocity=1 -> lower=-2.25 upper=0.78 effort=100 velocity=100
- joint LElbow: limit lower=-1.57 upper=1.0 effort=1 velocity=1 -> lower=-1.57 upper=1.0 effort=100 velocity=100
- joint LForearm: limit lower=-2.5 upper=0.0 effort=1 velocity=1 -> lower=-2.5 upper=0.0 effort=100 velocity=100
- joint LLeg_0: limit lower=-0.52 upper=0.87 effort=1 velocity=1 -> lower=-0.52 upper=0.87 effort=100 velocity=100
- joint LLeg_1: limit lower=-2.3 upper=0.52 effort=1 velocity=1 -> lower=-2.3 upper=0.52 effort=100 velocity=100
- joint LLeg_2: limit lower=-0.8 upper=0.8 effort=1 velocity=1 -> lower=-0.8 upper=0.8 effort=100 velocity=100
- joint LShin_0: limit lower=0.0 upper=2.6 effort=1 velocity=1 -> lower=0.0 upper=2.6 effort=100 velocity=100
- joint LWrist_0: limit lower=-1.5 upper=1.5 effort=1 velocity=1 -> lower=-1.5 upper=1.5 effort=100 velocity=100
- joint LWrist_1: limit lower=-0.35 upper=0.35 effort=1 velocity=1 -> lower=-0.35 upper=0.35 effort=100 velocity=100
- joint RAnkle_0: child RAnkleLink -> shin2rankle_1; limit lower=-0.78 upper=1.3 effort=1 velocity=1 -> lower=-0.78 upper=1.3 effort=100 velocity=100
- joint RArm_0: limit lower=-1.42 upper=1.57 effort=1 velocity=1 -> lower=-1.42 upper=1.57 effort=100 velocity=100
- joint RArm_1: limit lower=-1.2 upper=1.2 effort=1 velocity=1 -> lower=-1.2 upper=1.2 effort=100 velocity=100
- joint RArm_2: limit lower=-2.25 upper=0.78 effort=1 velocity=1 -> lower=-2.25 upper=0.78 effort=100 velocity=100
- joint RElbow: limit lower=-1.57 upper=1.0 effort=1 velocity=1 -> lower=-1.57 upper=1.0 effort=100 velocity=100
- joint RForearm: limit lower=-2.5 upper=0.0 effort=1 velocity=1 -> lower=0.0 upper=2.5 effort=100 velocity=100
- joint RLeg_0: limit lower=-0.87 upper=0.52 effort=1 velocity=1 -> lower=-0.87 upper=0.52 effort=100 velocity=100
- joint RLeg_1: limit lower=-2.3 upper=0.52 effort=1 velocity=1 -> lower=-2.3 upper=0.52 effort=100 velocity=100
- joint RLeg_2: limit lower=-0.8 upper=0.8 effort=1 velocity=1 -> lower=-0.8 upper=0.8 effort=100 velocity=100
- joint RShin_0: limit lower=0.0 upper=2.6 effort=1 velocity=1 -> lower=0.0 upper=2.6 effort=100 velocity=100
- joint RWrist_0: limit lower=-1.5 upper=1.5 effort=1 velocity=1 -> lower=-1.5 upper=1.5 effort=100 velocity=100
- joint RWrist_1: limit lower=-0.35 upper=0.35 effort=1 velocity=1 -> lower=-0.35 upper=0.35 effort=100 velocity=100
- joint Torso_0: limit lower=-0.65 upper=0.65 effort=1 velocity=1 -> lower=-0.65 upper=0.65 effort=100 velocity=100
- joint Torso_1: limit lower=-0.55 upper=2.9 effort=1 velocity=1 -> lower=-0.55 upper=2.9 effort=100 velocity=100
- joint Torso_2: limit lower=-0.7 upper=0.7 effort=1 velocity=1 -> lower=-0.7 upper=0.7 effort=100 velocity=100

Commit message: Changed free-flyer position, fixed arm joints limits

File: urdf/human.urdf (robot description, URDF)
Before this commit: robot HUMAN, 34 links, 33 joints
Joints:
- joint LArm_2: limit lower=-2.25 upper=0.78 effort=100 velocity=100 -> lower=-2.8 upper=0.9 effort=100 velocity=100
- joint RArm_2: limit lower=-2.25 upper=0.78 effort=100 velocity=100 -> lower=-0.9 upper=2.8 effort=100 velocity=100
- joint base: origin xyz=0 0 0.987 rpy=0 0 0 -> xyz=0 0 0 rpy=0 0 0

Commit message: Added gripper type hand joints system to main URDF
* Fixed some hand joint names and rotation axes
* Removed all other URDF files

File: urdf/human.urdf (robot description, URDF)
Before this commit: robot HUMAN, 34 links, 33 joints
Links:
- added link LHandBaby1Link, mass 0.0182; collision mesh filename=package://human_description/meshes/LBaby1stPhalange.dae; visual mesh filename=package://human_description/meshes/LBaby1stPhalange.dae
- added link LHandBaby2Link, mass 0.0182; collision mesh filename=package://human_description/meshes/LBaby2ndPhalange.dae; visual mesh filename=package://human_description/meshes/LBaby2ndPhalange.dae
- added link LHandBaby3Link, mass 0.0182; collision mesh filename=package://human_description/meshes/LBaby3rdPhalange.dae; visual mesh filename=package://human_description/meshes/LBaby3rdPhalange.dae
- added link LHandIndex1Link, mass 0.0182; collision mesh filename=package://human_description/meshes/LIndex1stPhalange.dae; visual mesh filename=package://human_description/meshes/LIndex1stPhalange.dae
- added link LHandIndex2Link, mass 0.0182; collision mesh filename=package://human_description/meshes/LIndex2ndPhalange.dae; visual mesh filename=package://human_description/meshes/LIndex2ndPhalange.dae
- added link LHandIndex3Link, mass 0.0182; collision mesh filename=package://human_description/meshes/LIndex3rdPhalange.dae; visual mesh filename=package://human_description/meshes/LIndex3rdPhalange.dae
- added link LHandMiddle1Link, mass 0.0182; collision mesh filename=package://human_description/meshes/LMiddle1stPhalange.dae; visual mesh filename=package://human_description/meshes/LMiddle1stPhalange.dae
- added link LHandMiddle2Link, mass 0.0182; collision mesh filename=package://human_description/meshes/LMiddle2ndPhalange.dae; visual mesh filename=package://human_description/meshes/LMiddle2ndPhalange.dae
- added link LHandMiddle3Link, mass 0.0182; collision mesh filename=package://human_description/meshes/LMiddle3rdPhalange.dae; visual mesh filename=package://human_description/meshes/LMiddle3rdPhalange.dae
- added link LHandRing1Link, mass 0.0182; collision mesh filename=package://human_description/meshes/LRing1stPhalange.dae; visual mesh filename=package://human_description/meshes/LRing1stPhalange.dae
- added link LHandRing2Link, mass 0.0182; collision mesh filename=package://human_description/meshes/LRing2ndPhalange.dae; visual mesh filename=package://human_description/meshes/LRing2ndPhalange.dae
- added link LHandRing3Link, mass 0.0182; collision mesh filename=package://human_description/meshes/LRing3rdPhalange.dae; visual mesh filename=package://human_description/meshes/LRing3rdPhalange.dae
- added link LHandThumb0Link, mass 0.0182; collision mesh filename=package://human_description/meshes/LThumb0thPhalange.dae; visual mesh filename=package://human_description/meshes/LThumb0thPhalange.dae
- added link LHandThumb1Link, mass 0.0182; collision mesh filename=package://human_description/meshes/LThumb1stPhalange.dae; visual mesh filename=package://human_description/meshes/LThumb1stPhalange.dae
- added link LHandThumb2Link, mass 0.0182; collision mesh filename=package://human_description/meshes/LThumb2ndPhalange.dae; visual mesh filename=package://human_description/meshes/LThumb2ndPhalange.dae
- added link RHandBaby1Link, mass 0.0182; collision mesh filename=package://human_description/meshes/RBaby1stPhalange.dae; visual mesh filename=package://human_description/meshes/RBaby1stPhalange.dae
- added link RHandBaby2Link, mass 0.0182; collision mesh filename=package://human_description/meshes/RBaby2ndPhalange.dae; visual mesh filename=package://human_description/meshes/RBaby2ndPhalange.dae
- added link RHandBaby3Link, mass 0.0182; collision mesh filename=package://human_description/meshes/RBaby3rdPhalange.dae; visual mesh filename=package://human_description/meshes/RBaby3rdPhalange.dae
- added link RHandIndex1Link, mass 0.0182; collision mesh filename=package://human_description/meshes/RIndex1stPhalange.dae; visual mesh filename=package://human_description/meshes/RIndex1stPhalange.dae
- added link RHandIndex2Link, mass 0.0182; collision mesh filename=package://human_description/meshes/RIndex2ndPhalange.dae; visual mesh filename=package://human_description/meshes/RIndex2ndPhalange.dae
- added link RHandIndex3Link, mass 0.0182; collision mesh filename=package://human_description/meshes/RIndex3rdPhalange.dae; visual mesh filename=package://human_description/meshes/RIndex3rdPhalange.dae
- added link RHandMiddle1Link, mass 0.0182; collision mesh filename=package://human_description/meshes/RMiddle1stPhalange.dae; visual mesh filename=package://human_description/meshes/RMiddle1stPhalange.dae
- added link RHandMiddle2Link, mass 0.0182; collision mesh filename=package://human_description/meshes/RMiddle2ndPhalange.dae; visual mesh filename=package://human_description/meshes/RMiddle2ndPhalange.dae
- added link RHandMiddle3Link, mass 0.0182; collision mesh filename=package://human_description/meshes/RMiddle3rdPhalange.dae; visual mesh filename=package://human_description/meshes/RMiddle3rdPhalange.dae
- added link RHandRing1Link, mass 0.0182; collision mesh filename=package://human_description/meshes/RRing1stPhalange.dae; visual mesh filename=package://human_description/meshes/RRing1stPhalange.dae
- added link RHandRing2Link, mass 0.0182; collision mesh filename=package://human_description/meshes/RRing2ndPhalange.dae; visual mesh filename=package://human_description/meshes/RRing2ndPhalange.dae
- added link RHandRing3Link, mass 0.0182; collision mesh filename=package://human_description/meshes/RRing3rdPhalange.dae; visual mesh filename=package://human_description/meshes/RRing3rdPhalange.dae
- added link RHandThumb0Link, mass 0.0182; collision mesh filename=package://human_description/meshes/RThumb0thPhalange.dae; visual mesh filename=package://human_description/meshes/RThumb0thPhalange.dae
- added link RHandThumb1Link, mass 0.0182; collision mesh filename=package://human_description/meshes/RThumb1stPhalange.dae; visual mesh filename=package://human_description/meshes/RThumb1stPhalange.dae
- added link RHandThumb2Link, mass 0.0182; collision mesh filename=package://human_description/meshes/RThumb2ndPhalange.dae; visual mesh filename=package://human_description/meshes/RThumb2ndPhalange.dae
- added link l_gripper, mass 2e-06
- added link r_gripper, mass 2e-06
- link forearm2lwrist_1: geometry 
- link forearm2rwrist_1: geometry 
- link hip2torso_1: geometry 
- link hip2torso_2: geometry 
- link shin2lankle_1: geometry 
- link shin2rankle_1: geometry 
- link torso2head_1: geometry 
- link torso2head_2: geometry 
- link torso2lleg_1: geometry 
- link torso2lleg_2: geometry 
- link torso2lshoulder_1: geometry 
- link torso2lshoulder_2: geometry 
- link torso2rleg_1: geometry 
- link torso2rleg_2: geometry 
- link torso2rshoulder_1: geometry 
- link torso2rshoulder_2: geometry 
Joints:
- added joint LHand: type revolute, parent LHandLink, child l_gripper, origin xyz=0.025 0 0 rpy=0 0 0, axis 1.0 0 0, limit lower=0 upper=1 effort=0.144 velocity=12.56
- added joint LHandBabyLink1: type continuous, parent LHandLink, child LHandBaby1Link, origin xyz=-0.015 0.079 -0.022 rpy=0.0 0.0 0.0, axis -1 0 0, mimic joint=LHand multiplier=0.8 offset=0
- added joint LHandBabyLink2: type continuous, parent LHandBaby1Link, child LHandBaby2Link, origin xyz=-0.0 0.02 0.0 rpy=0.0 0.0 0.0, axis -1 0 0, mimic joint=LHand multiplier=0.8 offset=0
- added joint LHandBabyLink3: type continuous, parent LHandBaby2Link, child LHandBaby3Link, origin xyz=-0.0 0.02 0.0 rpy=0.0 0.0 0.0, axis -1 0 0, mimic joint=LHand multiplier=0.8 offset=0
- added joint LHandIndexLink1: type continuous, parent LHandLink, child LHandIndex1Link, origin xyz=0.0425 0.078 -0.01 rpy=0.0 0.0 0.0, axis -1 0 0, mimic joint=LHand multiplier=0.8 offset=0
- added joint LHandIndexLink2: type continuous, parent LHandIndex1Link, child LHandIndex2Link, origin xyz=-0.0 0.035 0.0 rpy=0.0 0.0 0.0, axis -1 0 0, mimic joint=LHand multiplier=0.8 offset=0
- added joint LHandIndexLink3: type continuous, parent LHandIndex2Link, child LHandIndex3Link, origin xyz=-0.0 0.022 0.0 rpy=0.0 0.0 0.0, axis -1 0 0, mimic joint=LHand multiplier=0.8 offset=0
- added joint LHandMiddleLink1: type continuous, parent LHandLink, child LHandMiddle1Link, origin xyz=0.02 0.09 -0.01 rpy=0.0 0.0 0.0, axis -1 0 0, mimic joint=LHand multiplier=0.8 offset=0
- added joint LHandMiddleLink2: type continuous, parent LHandMiddle1Link, child LHandMiddle2Link, origin xyz=-0.0 0.028 0.0 rpy=0.0 0.0 0.0, axis -1 0 0, mimic joint=LHand multiplier=0.8 offset=0
- added joint LHandMiddleLink3: type continuous, parent LHandMiddle2Link, child LHandMiddle3Link, origin xyz=-0.0 0.025 0.0 rpy=0.0 0.0 0.0, axis -1 0 0, mimic joint=LHand multiplier=0.8 offset=0
- added joint LHandRingLink1: type continuous, parent LHandLink, child LHandRing1Link, origin xyz=-0.001 0.085 -0.01 rpy=0.0 0.0 0.0, axis -1 0 0, mimic joint=LHand multiplier=0.8 offset=0
- added joint LHandRingLink2: type continuous, parent LHandRing1Link, child LHandRing2Link, origin xyz=-0.0 0.0225 0.0 rpy=0.0 0.0 0.0, axis -1 0 0, mimic joint=LHand multiplier=0.8 offset=0
- added joint LHandRingLink3: type continuous, parent LHandRing2Link, child LHandRing3Link, origin xyz=-0.0 0.028 0.0 rpy=0.0 0.0 0.0, axis -1 0 0, mimic joint=LHand multiplier=0.8 offset=0
- added joint LHandThumbLink1: type continuous, parent LHandLink, child LHandThumb0Link, origin xyz=0.025 0.016 -0.016 rpy=0.5 0.0 0.7, axis 0 1 0, mimic joint=LHand multiplier=0.3 offset=0
- added joint LHandThumbLink2: type continuous, parent LHandThumb0Link, child LHandThumb1Link, origin xyz=0.045 0.0 0.0 rpy=0.0 0.0 0.0, axis 0 1 0, mimic joint=LHand multiplier=0.8 offset=0
- added joint LHandThumbLink3: type continuous, parent LHandThumb1Link, child LHandThumb2Link, origin xyz=0.026 0.0 0.0 rpy=0.0 0.0 0.0, axis 0 1 0, mimic joint=LHand multiplier=0.8 offset=0
- added joint RHand: type revolute, parent RHandLink, child r_gripper, origin xyz=0.025 0 0 rpy=0 0 0, axis 1.0 0 0, limit lower=0 upper=1 effort=0.144 velocity=12.56
- added joint RHandBabyLink1: type continuous, parent RHandLink, child RHandBaby1Link, origin xyz=-0.015 -0.079 -0.022 rpy=0.0 0.0 0.0, axis 1 0 0, mimic joint=RHand multiplier=0.8 offset=0
- added joint RHandBabyLink2: type continuous, parent RHandBaby1Link, child RHandBaby2Link, origin xyz=-0.0 -0.02 0.0 rpy=0.0 0.0 0.0, axis 1 0 0, mimic joint=RHand multiplier=0.8 offset=0
- added joint RHandBabyLink3: type continuous, parent RHandBaby2Link, child RHandBaby3Link, origin xyz=-0.0 -0.02 0.0 rpy=0.0 0.0 0.0, axis 1 0 0, mimic joint=RHand multiplier=0.8 offset=0
- added joint RHandIndexLink1: type continuous, parent RHandLink, child RHandIndex1Link, origin xyz=0.0425 -0.078 -0.01 rpy=0.0 0.0 0.0, axis 1 0 0, mimic joint=RHand multiplier=0.8 offset=0
- added joint RHandIndexLink2: type continuous, parent RHandIndex1Link, child RHandIndex2Link, origin xyz=-0.0 -0.035 0.0 rpy=0.0 0.0 0.0, axis 1 0 0, mimic joint=RHand multiplier=0.8 offset=0
- added joint RHandIndexLink3: type continuous, parent RHandIndex2Link, child RHandIndex3Link, origin xyz=-0.0 -0.022 0.0 rpy=0.0 0.0 0.0, axis 1 0 0, mimic joint=RHand multiplier=0.8 offset=0
- added joint RHandMiddleLink1: type continuous, parent RHandLink, child RHandMiddle1Link, origin xyz=0.02 -0.09 -0.01 rpy=0.0 0.0 0.0, axis 1 0 0, mimic joint=RHand multiplier=0.8 offset=0
- added joint RHandMiddleLink2: type continuous, parent RHandMiddle1Link, child RHandMiddle2Link, origin xyz=-0.0 -0.028 0.0 rpy=0.0 0.0 0.0, axis 1 0 0, mimic joint=RHand multiplier=0.8 offset=0
- added joint RHandMiddleLink3: type continuous, parent RHandMiddle2Link, child RHandMiddle3Link, origin xyz=-0.0 -0.025 0.0 rpy=0.0 0.0 0.0, axis 1 0 0, mimic joint=RHand multiplier=0.8 offset=0
- added joint RHandRingLink1: type continuous, parent RHandLink, child RHandRing1Link, origin xyz=-0.001 -0.085 -0.01 rpy=0.0 0.0 0.0, axis 1 0 0, mimic joint=RHand multiplier=0.8 offset=0
- added joint RHandRingLink2: type continuous, parent RHandRing1Link, child RHandRing2Link, origin xyz=-0.0 -0.0225 0.0 rpy=0.0 0.0 0.0, axis 1 0 0, mimic joint=RHand multiplier=0.8 offset=0
- added joint RHandRingLink3: type continuous, parent RHandRing2Link, child RHandRing3Link, origin xyz=-0.0 -0.028 0.0 rpy=0.0 0.0 0.0, axis 1 0 0, mimic joint=RHand multiplier=0.8 offset=0
- added joint RHandThumbLink1: type continuous, parent RHandLink, child RHandThumb0Link, origin xyz=0.025 -0.016 -0.016 rpy=-0.5 0.0 -0.7, axis 0 1 0, mimic joint=RHand multiplier=0.3 offset=0
- added joint RHandThumbLink2: type continuous, parent RHandThumb0Link, child RHandThumb1Link, origin xyz=0.045 0.0 0.0 rpy=0.0 0.0 0.0, axis 0 1 0, mimic joint=RHand multiplier=0.8 offset=0
- added joint RHandThumbLink3: type continuous, parent RHandThumb1Link, child RHandThumb2Link, origin xyz=0.026 0.0 0.0 rpy=0.0 0.0 0.0, axis 0 1 0, mimic joint=RHand multiplier=0.8 offset=0
