Commit message: [mujoco] Basic options to convert to mujoco

File: urdf/human.urdf (robot description, URDF)
Before this commit: robot HUMAN, 66 links, 65 joints
Links:
- link HeadLink: geometry collision mesh filename=package://human_description/meshes/HeadLinkFull.stl; visual mesh filename=package://human_description/meshes/HeadLinkFull.stl
- link HipsLink: geometry collision mesh filename=package://human_description/meshes/HipsLinkFull.stl; visual mesh filename=package://human_description/meshes/HipsLinkFull.stl
- link LAnkleLink: geometry collision mesh filename=package://human_description/meshes/LAnkleLinkFull.stl; visual mesh filename=package://human_description/meshes/LAnkleLinkFull.stl
- link LArmLink: geometry collision mesh filename=package://human_description/meshes/LArmLinkFull.stl; visual mesh filename=package://human_description/meshes/LArmLinkFull.stl
- link LElbowLink: geometry collision mesh filename=package://human_description/meshes/LElbowLink.stl; visual mesh filename=package://human_description/meshes/LElbowLink.stl
- link LForearmLink: geometry collision mesh filename=package://human_description/meshes/LForearmLink.stl; visual mesh filename=package://human_description/meshes/LForearmLink.stl
- link LHandBaby1Link: geometry collision mesh filename=package://human_description/meshes/LBaby1stPhalange.stl; visual mesh filename=package://human_description/meshes/LBaby1stPhalange.stl
- link LHandBaby2Link: geometry collision mesh filename=package://human_description/meshes/LBaby2ndPhalange.stl; visual mesh filename=package://human_description/meshes/LBaby2ndPhalange.stl
- link LHandBaby3Link: geometry collision mesh filename=package://human_description/meshes/LBaby3rdPhalange.stl; visual mesh filename=package://human_description/meshes/LBaby3rdPhalange.stl
- link LHandIndex1Link: geometry collision mesh filename=package://human_description/meshes/LIndex1stPhalange.stl; visual mesh filename=package://human_description/meshes/LIndex1stPhalange.stl
- link LHandIndex2Link: geometry collision mesh filename=package://human_description/meshes/LIndex2ndPhalange.stl; visual mesh filename=package://human_description/meshes/LIndex2ndPhalange.stl
- link LHandIndex3Link: geometry collision mesh filename=package://human_description/meshes/LIndex3rdPhalange.stl; visual mesh filename=package://human_description/meshes/LIndex3rdPhalange.stl
- link LHandLink: geometry collision mesh filename=package://human_description/meshes/LWrist.stl; visual mesh filename=package://human_description/meshes/LWrist.stl
- link LHandMiddle1Link: geometry collision mesh filename=package://human_description/meshes/LMiddle1stPhalange.stl; visual mesh filename=package://human_description/meshes/LMiddle1stPhalange.stl
- link LHandMiddle2Link: geometry collision mesh filename=package://human_description/meshes/LMiddle2ndPhalange.stl; visual mesh filename=package://human_description/meshes/LMiddle2ndPhalange.stl
- link LHandMiddle3Link: geometry collision mesh filename=package://human_description/meshes/LMiddle3rdPhalange.stl; visual mesh filename=package://human_description/meshes/LMiddle3rdPhalange.stl
- link LHandRing1Link: geometry collision mesh filename=package://human_description/meshes/LRing1stPhalange.stl; visual mesh filename=package://human_description/meshes/LRing1stPhalange.stl
- link LHandRing2Link: geometry collision mesh filename=package://human_description/meshes/LRing2ndPhalange.stl; visual mesh filename=package://human_description/meshes/LRing2ndPhalange.stl
- link LHandRing3Link: geometry collision mesh filename=package://human_description/meshes/LRing3rdPhalange.stl; visual mesh filename=package://human_description/meshes/LRing3rdPhalange.stl
- link LHandThumb0Link: geometry collision mesh filename=package://human_description/meshes/LThumb0thPhalange.stl; visual mesh filename=package://human_description/meshes/LThumb0thPhalange.stl
- link LHandThumb1Link: geometry collision mesh filename=package://human_description/meshes/LThumb1stPhalange.stl; visual mesh filename=package://human_description/meshes/LThumb1stPhalange.stl
- link LHandThumb2Link: geometry collision mesh filename=package://human_description/meshes/LThumb2ndPhalange.stl; visual mesh filename=package://human_description/meshes/LThumb2ndPhalange.stl
- link LLegLink: geometry collision mesh filename=package://human_description/meshes/LLegLink.stl; visual mesh filename=package://human_description/meshes/LLegLink.stl
- link LShinLink: geometry collision mesh filename=package://human_description/meshes/LShinLink.stl; visual mesh filename=package://human_description/meshes/LShinLink.stl
- link RAnkleLink: geometry collision mesh filename=package://human_description/meshes/RAnkleLinkFull.stl; visual mesh filename=package://human_description/meshes/RAnkleLinkFull.stl
- link RArmLink: geometry collision mesh filename=package://human_description/meshes/RArmLinkFull.stl; visual mesh filename=package://human_description/meshes/RArmLinkFull.stl
- link RElbowLink: geometry collision mesh filename=package://human_description/meshes/RElbowLink.stl; visual mesh filename=package://human_description/meshes/RElbowLink.stl
- link RForearmLink: geometry collision mesh filename=package://human_description/meshes/RForearmLink.stl; visual mesh filename=package://human_description/meshes/RForearmLink.stl
- link RHandBaby1Link: geometry collision mesh filename=package://human_description/meshes/RBaby1stPhalange.stl; visual mesh filename=package://human_description/meshes/RBaby1stPhalange.stl
- link RHandBaby2Link: geometry collision mesh filename=package://human_description/meshes/RBaby2ndPhalange.stl; visual mesh filename=package://human_description/meshes/RBaby2ndPhalange.stl
- link RHandBaby3Link: geometry collision mesh filename=package://human_description/meshes/RBaby3rdPhalange.stl; visual mesh filename=package://human_description/meshes/RBaby3rdPhalange.stl
- link RHandIndex1Link: geometry collision mesh filename=package://human_description/meshes/RIndex1stPhalange.stl; visual mesh filename=package://human_description/meshes/RIndex1stPhalange.stl
- link RHandIndex2Link: geometry collision mesh filename=package://human_description/meshes/RIndex2ndPhalange.stl; visual mesh filename=package://human_description/meshes/RIndex2ndPhalange.stl
- link RHandIndex3Link: geometry collision mesh filename=package://human_description/meshes/RIndex3rdPhalange.stl; visual mesh filename=package://human_description/meshes/RIndex3rdPhalange.stl
- link RHandLink: geometry collision mesh filename=package://human_description/meshes/RWrist.stl; visual mesh filename=package://human_description/meshes/RWrist.stl
- link RHandMiddle1Link: geometry collision mesh filename=package://human_description/meshes/RMiddle1stPhalange.stl; visual mesh filename=package://human_description/meshes/RMiddle1stPhalange.stl
- link RHandMiddle2Link: geometry collision mesh filename=package://human_description/meshes/RMiddle2ndPhalange.stl; visual mesh filename=package://human_description/meshes/RMiddle2ndPhalange.stl
- link RHandMiddle3Link: geometry collision mesh filename=package://human_description/meshes/RMiddle3rdPhalange.stl; visual mesh filename=package://human_description/meshes/RMiddle3rdPhalange.stl
- link RHandRing1Link: geometry collision mesh filename=package://human_description/meshes/RRing1stPhalange.stl; visual mesh filename=package://human_description/meshes/RRing1stPhalange.stl
- link RHandRing2Link: geometry collision mesh filename=package://human_description/meshes/RRing2ndPhalange.stl; visual mesh filename=package://human_description/meshes/RRing2ndPhalange.stl
- link RHandRing3Link: geometry collision mesh filename=package://human_description/meshes/RRing3rdPhalange.stl; visual mesh filename=package://human_description/meshes/RRing3rdPhalange.stl
- link RHandThumb0Link: geometry collision mesh filename=package://human_description/meshes/RThumb0thPhalange.stl; visual mesh filename=package://human_description/meshes/RThumb0thPhalange.stl
- link RHandThumb1Link: geometry collision mesh filename=package://human_description/meshes/RThumb1stPhalange.stl; visual mesh filename=package://human_description/meshes/RThumb1stPhalange.stl
- link RHandThumb2Link: geometry collision mesh filename=package://human_description/meshes/RThumb2ndPhalange.stl; visual mesh filename=package://human_description/meshes/RThumb2ndPhalange.stl
- link RLegLink: geometry collision mesh filename=package://human_description/meshes/RLegLink.stl; visual mesh filename=package://human_description/meshes/RLegLink.stl
- link RShinLink: geometry collision mesh filename=package://human_description/meshes/RShinLink.stl; visual mesh filename=package://human_description/meshes/RShinLink.stl
- link TorsoLink: geometry collision mesh filename=package://human_description/meshes/TorsoLinkFull.stl; visual mesh filename=package://human_description/meshes/TorsoLinkFull.stl
